File: hardware/ultrasonic-distance.kicad_sch (KiCad schematic)
At the start: 5 parts, among them U1 ATmega328-P, Y1 ABL-16.000MHZ-B2

Commit message: Mostly footprint items
Parts:
- added J1: USB_C_Receptacle_USB2.0_16P, Connector_USB:USB_C_Receptacle_GCT_USB4110, symbol Connector:USB_C_Receptacle_USB2.0_16P
- C1, C2: footprint (none) -> Library:CAP_K220J15C0GF53L2_VIS
- C3: footprint (none) -> Library:U1-S_NCH
- Y1: footprint ABL-16.000MHZ-B2:XTAL_HC49P488W46L1150T500H350 -> Library:XTAL_HC49P488W46L1150T500H350
Connections:
- net GND: now also J1.A1 (GND), J1.A12 (GND), J1.B1 (GND), J1.B12 (GND), J1.S1 (SHIELD)
- new net: J1.A4 (VBUS), J1.A9 (VBUS), J1.B4 (VBUS), J1.B9 (VBUS)
Other:
- moved on the sheet: C1, C2, C3, U1, Y1
